Commit message: update g1

File: unitree_g1_ros1/urdf/g1_29dof_with_hand_rev_1_0.urdf (robot description, URDF)
Before this commit: robot g1_29dof_with_hand_rev_1_0, 53 links, 52 joints
Links:
- removed link left_hand_index_0_link
- removed link left_hand_index_1_link
- removed link left_hand_middle_0_link
- removed link left_hand_middle_1_link
- removed link left_hand_palm_link
- removed link left_hand_thumb_0_link
- removed link left_hand_thumb_1_link
- removed link left_hand_thumb_2_link
- removed link right_hand_index_0_link
- removed link right_hand_index_1_link
- removed link right_hand_middle_0_link
- removed link right_hand_middle_1_link
- removed link right_hand_palm_link
- removed link right_hand_thumb_0_link
- removed link right_hand_thumb_1_link
- removed link right_hand_thumb_2_link
- added link L_hand_base_link, mass 0.14143; collision mesh filename=package://unitree_g1_ros2/meshes/L_hand_base_link.STL; visual mesh filename=package://unitree_g1_ros2/meshes/L_hand_base_link.STL
- added link L_index_distal, mass 0.0045682; collision mesh filename=package://unitree_g1_ros2/meshes/L_index_distal.STL; visual mesh filename=package://unitree_g1_ros2/meshes/L_index_distal.STL
- added link L_index_proximal, mass 0.0042405; collision mesh filename=package://unitree_g1_ros2/meshes/L_index_proximal.STL; visual mesh filename=package://unitree_g1_ros2/meshes/L_index_proximal.STL
- added link L_middle_distal, mass 0.0050397; collision mesh filename=package://unitree_g1_ros2/meshes/L_middle_distal.STL; visual mesh filename=package://unitree_g1_ros2/meshes/L_middle_distal.STL
- added link L_middle_proximal, mass 0.0042405; collision mesh filename=package://unitree_g1_ros2/meshes/L_middle_proximal.STL; visual mesh filename=package://unitree_g1_ros2/meshes/L_middle_proximal.STL
- added link L_pinky_distal, mass 0.0036036; collision mesh filename=package://unitree_g1_ros2/meshes/L_pinky_distal.STL; visual mesh filename=package://unitree_g1_ros2/meshes/L_pinky_distal.STL
- added link L_pinky_proximal, mass 0.0042405; collision mesh filename=package://unitree_g1_ros2/meshes/L_pinky_proximal.STL; visual mesh filename=package://unitree_g1_ros2/meshes/L_pinky_proximal.STL
- added link L_ring_distal, mass 0.0045682; collision mesh filename=package://unitree_g1_ros2/meshes/L_ring_distal.STL; visual mesh filename=package://unitree_g1_ros2/meshes/L_ring_distal.STL
- added link L_ring_proximal, mass 0.0042405; collision mesh filename=package://unitree_g1_ros2/meshes/L_ring_proximal.STL; visual mesh filename=package://unitree_g1_ros2/meshes/L_ring_proximal.STL
- added link L_thumb_distal, mass 0.003344; collision mesh filename=package://unitree_g1_ros2/meshes/L_thumb_distal.STL; visual mesh filename=package://unitree_g1_ros2/meshes/L_thumb_distal.STL
- added link L_thumb_intermediate, mass 0.0037844; collision mesh filename=package://unitree_g1_ros2/meshes/L_thumb_intermediate.STL; visual mesh filename=package://unitree_g1_ros2/meshes/L_thumb_intermediate.STL
- added link L_thumb_proximal, mass 0.0066101; collision mesh filename=package://unitree_g1_ros2/meshes/L_thumb_proximal.STL; visual mesh filename=package://unitree_g1_ros2/meshes/L_thumb_proximal.STL
- added link L_thumb_proximal_base, mass 0.0018869; collision mesh filename=package://unitree_g1_ros2/meshes/L_thumb_proximal_base.STL; visual mesh filename=package://unitree_g1_ros2/meshes/L_thumb_proximal_base.STL
- added link R_hand_base_link, mass 0.14143; collision mesh filename=package://unitree_g1_ros2/meshes/R_hand_base_link.STL; visual mesh filename=package://unitree_g1_ros2/meshes/R_hand_base_link.STL
- added link R_index_distal, mass 0.0045683; collision mesh filename=package://unitree_g1_ros2/meshes/R_index_distal.STL; visual mesh filename=package://unitree_g1_ros2/meshes/R_index_distal.STL
- added link R_index_proximal, mass 0.0042403; collision mesh filename=package://unitree_g1_ros2/meshes/R_index_proximal.STL; visual mesh filename=package://unitree_g1_ros2/meshes/R_index_proximal.STL
- added link R_middle_distal, mass 0.0050396; collision mesh filename=package://unitree_g1_ros2/meshes/R_middle_distal.STL; visual mesh filename=package://unitree_g1_ros2/meshes/R_middle_distal.STL
- added link R_middle_proximal, mass 0.0042403; collision mesh filename=package://unitree_g1_ros2/meshes/R_middle_proximal.STL; visual mesh filename=package://unitree_g1_ros2/meshes/R_middle_proximal.STL
- added link R_pinky_distal, mass 0.0035996; collision mesh filename=package://unitree_g1_ros2/meshes/R_pinky_distal.STL; visual mesh filename=package://unitree_g1_ros2/meshes/R_pinky_distal.STL
- added link R_pinky_proximal, mass 0.0042403; collision mesh filename=package://unitree_g1_ros2/meshes/R_pinky_proximal.STL; visual mesh filename=package://unitree_g1_ros2/meshes/R_pinky_proximal.STL
- added link R_ring_distal, mass 0.0045683; collision mesh filename=package://unitree_g1_ros2/meshes/R_ring_distal.STL; visual mesh filename=package://unitree_g1_ros2/meshes/R_ring_distal.STL
- added link R_ring_proximal, mass 0.0042403; collision mesh filename=package://unitree_g1_ros2/meshes/R_ring_proximal.STL; visual mesh filename=package://unitree_g1_ros2/meshes/R_ring_proximal.STL
- added link R_thumb_distal, mass 0.0033441; collision mesh filename=package://unitree_g1_ros2/meshes/R_thumb_distal.STL; visual mesh filename=package://unitree_g1_ros2/meshes/R_thumb_distal.STL
- added link R_thumb_intermediate, mass 0.0037847; collision mesh filename=package://unitree_g1_ros2/meshes/R_thumb_intermediate.STL; visual mesh filename=package://unitree_g1_ros2/meshes/R_thumb_intermediate.STL
- added link R_thumb_proximal, mass 0.0066075; collision mesh filename=package://unitree_g1_ros2/meshes/R_thumb_proximal.STL; visual mesh filename=package://unitree_g1_ros2/meshes/R_thumb_proximal.STL
- added link R_thumb_proximal_base, mass 0.0018869; collision mesh filename=package://unitree_g1_ros2/meshes/R_thumb_proximal_base.STL; visual mesh filename=package://unitree_g1_ros2/meshes/R_thumb_proximal_base.STL
- link head_link: geometry collision mesh filename=package://unitree_g1_ros2/meshes/head_link.STL; visual mesh filename=package://unitree_g1_ros2/meshes/head_link.STL
- link left_ankle_pitch_link: geometry collision mesh filename=package://unitree_g1_ros2/meshes/left_ankle_pitch_link.STL; visual mesh filename=package://unitree_g1_ros2/meshes/left_ankle_pitch_link.STL
- link left_ankle_roll_link: geometry collision sphere radius=0.005; collision sphere radius=0.005
- link left_elbow_link: geometry collision mesh filename=package://unitree_g1_ros2/meshes/left_elbow_link.STL; visual mesh filename=package://unitree_g1_ros2/meshes/left_elbow_link.STL
- link left_hip_pitch_link: geometry collision mesh filename=package://unitree_g1_ros2/meshes/left_hip_pitch_link.STL; visual mesh filename=package://unitree_g1_ros2/meshes/left_hip_pitch_link.STL
- link left_hip_roll_link: geometry collision mesh filename=package://unitree_g1_ros2/meshes/left_hip_roll_link.STL; visual mesh filename=package://unitree_g1_ros2/meshes/left_hip_roll_link.STL
- link left_hip_yaw_link: geometry collision mesh filename=package://unitree_g1_ros2/meshes/left_hip_yaw_link.STL; visual mesh filename=package://unitree_g1_ros2/meshes/left_hip_yaw_link.STL
- link left_knee_link: geometry collision mesh filename=package://unitree_g1_ros2/meshes/left_knee_link.STL; visual mesh filename=package://unitree_g1_ros2/meshes/left_knee_link.STL
- link left_shoulder_pitch_link: geometry collision cylinder length=0.05 radius=0.03; visual mesh filename=package://unitree_g1_ros2/meshes/left_shoulder_pitch_link.S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
- link left_shoulder_roll_link: geometry collision cylinder length=0.03 radius=0.03; visual mesh filename=package://unitree_g1_ros2/meshes/left_shoulder_roll_link.STL
- link left_shoulder_yaw_link: geometry collision mesh filename=package://unitree_g1_ros2/meshes/left_shoulder_yaw_link.STL; visual mesh filename=package://unitree_g1_ros2/meshes/left_shoulder_yaw_link.STL
- link left_wrist_pitch_link: geometry collision mesh filename=package://unitree_g1_ros2/meshes/left_wrist_pitch_link.STL; visual mesh filename=package://unitree_g1_ros2/meshes/left_wrist_pitch_link.STL
- link left_wrist_roll_link: geometry collision mesh filename=package://unitree_g1_ros2/meshes/left_wrist_roll_link.STL; visual mesh filename=package://unitree_g1_ros2/meshes/left_wrist_roll_link.STL
- link left_wrist_yaw_link: geometry collision mesh filename=package://unitree_g1_ros2/meshes/left_wrist_yaw_link.STL; visual mesh filename=package://unitree_g1_ros2/meshes/left_wrist_yaw_link.STL
- link logo_link: geometry collision mesh filename=package://unitree_g1_ros2/meshes/logo_link.STL; visual mesh filename=package://unitree_g1_ros2/meshes/logo_link.STL
- link pelvis: geometry visual mesh filename=package://unitree_g1_ros2/meshes/pelvis.STL
- link pelvis_contour_link: geometry collision mesh filename=package://unitree_g1_ros2/meshes/pelvis_contour_link.STL; visual mesh filename=package://unitree_g1_ros2/meshes/pelvis_contour_link.STL
- link right_ankle_pitch_link: geometry collision mesh filename=package://unitree_g1_ros2/meshes/right_ankle_pitch_link.STL; visual mesh filename=package://unitree_g1_ros2/meshes/right_ankle_pitch_link.STL
- link right_ankle_roll_link: geometry collision sphere radius=0.005; collision sphere radius=0.005
- link right_elbow_link: geometry collision mesh filename=package://unitree_g1_ros2/meshes/right_elbow_link.STL; visual mesh filename=package://unitree_g1_ros2/meshes/right_elbow_link.STL
- link right_hip_pitch_link: geometry collision mesh filename=package://unitree_g1_ros2/meshes/right_hip_pitch_link.STL; visual mesh filename=package://unitree_g1_ros2/meshes/right_hip_pitch_link.STL
- link right_hip_roll_link: geometry collision mesh filename=package://unitree_g1_ros2/meshes/right_hip_roll_link.STL; visual mesh filename=package://unitree_g1_ros2/meshes/right_hip_roll_link.STL
- link right_hip_yaw_link: geometry collision mesh filename=package://unitree_g1_ros2/meshes/right_hip_yaw_link.STL; visual mesh filename=package://unitree_g1_ros2/meshes/right_hip_yaw_link.STL
- link right_knee_link: geometry collision mesh filename=package://unitree_g1_ros2/meshes/right_knee_link.STL; visual mesh filename=package://unitree_g1_ros2/meshes/right_knee_link.STL
- link right_shoulder_pitch_link: geometry collision cylinder length=0.05 radius=0.03; visual mesh filename=package://unitree_g1_ros2/meshes/right_shoulder_pitch_link.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
- link right_shoulder_roll_link: geometry collision cylinder length=0.03 radius=0.03; visual mesh filename=package://unitree_g1_ros2/meshes/right_shoulder_roll_link.S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
- link right_shoulder_yaw_link: geometry collision mesh filename=package://unitree_g1_ros2/meshes/right_shoulder_yaw_link.STL; visual mesh filename=package://unitree_g1_ros2/meshes/right_shoulder_yaw_link.STL
- link right_wrist_pitch_link: geometry collision mesh filename=package://unitree_g1_ros2/meshes/right_wrist_pitch_link.STL; visual mesh filename=package://unitree_g1_ros2/meshes/right_wrist_pitch_link.STL
- link right_wrist_roll_link: geometry collision mesh filename=package://unitree_g1_ros2/meshes/right_wrist_roll_link.STL; visual mesh filename=package://unitree_g1_ros2/meshes/right_wrist_roll_link.STL
- link right_wrist_yaw_link: geometry collision mesh filename=package://unitree_g1_ros2/meshes/right_wrist_yaw_link.STL; visual mesh filename=package://unitree_g1_ros2/meshes/right_wrist_yaw_link.STL
- link torso_link: geometry collision mesh filename=package://unitree_g1_ros2/meshes/torso_link_rev_1_0.STL; visual mesh filename=package://unitree_g1_ros2/meshes/torso_link_rev_1_0.STL
- link waist_roll_link: geometry visual mesh filename=package://unitree_g1_ros2/meshes/waist_roll_link_rev_1_0.STL
- link waist_yaw_link: geometry visual mesh filename=package://unitree_g1_ros2/meshes/waist_yaw_link_rev_1_0.STL
Joints:
- removed joint left_hand_index_0_joint
- removed joint left_hand_index_1_joint
- removed joint left_hand_middle_0_joint
- removed joint left_hand_middle_1_joint
- removed joint left_hand_thumb_0_joint
- removed joint left_hand_thumb_1_joint
- removed joint left_hand_thumb_2_joint
- removed joint right_hand_index_0_joint
- removed joint right_hand_index_1_joint
- removed joint right_hand_middle_0_joint
- removed joint right_hand_middle_1_joint
- removed joint right_hand_thumb_0_joint
- removed joint right_hand_thumb_1_joint
- removed joint right_hand_thumb_2_joint
- added joint L_index_DIP_joint: type revolute, parent L_index_proximal, child L_index_distal, origin xyz=0.0016538 0.030445 -0.010275 rpy=-0.079748 0 0, axis -1 0 0, limit lower=0 upper=1.527 effort=50 velocity=1, mimic joint=L_index_MCP_joint multiplier=1.1169 offset=0
- added joint L_index_MCP_joint: type revolute, parent L_hand_base_link, child L_index_proximal, origin xyz=0.018231106 0.000284483 -0.137012411 rpy=-1.3884 -0.034907 0, axis -1 0 0, limit lower=0 upper=1.41 effort=50 velocity=1
- added joint L_middle_DIP_joint: type revolute, parent L_middle_proximal, child L_middle_distal, origin xyz=0.0016698 0.030445 -0.010275 rpy=-0.111413 0 0, axis -1 0 0, limit lower=0 upper=1.527 effort=50 velocity=1, mimic joint=L_middle_MCP_joint multiplier=1.1169 offset=0
- added joint L_middle_MCP_joint: type revolute, parent L_hand_base_link, child L_middle_proximal, origin xyz=-0.001114894 0.000284483 -0.137012411 rpy=-1.3884 0 0, axis -1 0 0, limit lower=0 upper=1.41 effort=50 velocity=1
- added joint L_pinky_DIP_joint: type revolute, parent L_pinky_proximal, child L_pinky_distal, origin xyz=0 0.030445 -0.010275 rpy=-0.017691 0 0, axis -1 0 0, limit lower=0 upper=1.527 effort=50 velocity=1, mimic joint=L_pinky_MCP_joint multiplier=1.1169 offset=0
- added joint L_pinky_MCP_joint: type revolute, parent L_hand_base_link, child L_pinky_proximal, origin xyz=-0.044926894 0.000284483 -0.133672411 rpy=-1.3884 0.10472 0, axis -1 0 0, limit lower=0 upper=1.41 effort=50 velocity=1
- added joint L_ring_DIP_joint: type revolute, parent L_ring_proximal, child L_ring_distal, origin xyz=0.0015355 0.030445 -0.010275 rpy=-0.079748 0 0, axis -1 0 0, limit lower=0 upper=1.527 effort=50 velocity=1, mimic joint=L_ring_MCP_joint multiplier=1.1169 offset=0
- added joint L_ring_MCP_joint: type revolute, parent L_hand_base_link, child L_ring_proximal, origin xyz=-0.023084894 0.000284483 -0.136032411 rpy=-1.3884 0.05236 0, axis -1 0 0, limit lower=0 upper=1.41 effort=50 velocity=1
- added joint L_thumb_DIP_joint: type revolute, parent L_thumb_intermediate, child L_thumb_distal, origin xyz=0 0.022558 0.0020717 rpy=0.011642 0 0, axis -1 0 0, limit lower=0 upper=0.2775 effort=50 velocity=1, mimic joint=L_thumb_PIP_joint multiplier=0.7508 offset=0
- added joint L_thumb_MCP_joint1: type revolute, parent L_hand_base_link, child L_thumb_proximal_base, origin xyz=0.020450106 -0.016955517 -0.055202411 rpy=-1.5708 0 2.9722026, axis 0 1 0, limit lower=0 upper=1.096 effort=50 velocity=1
- added joint L_thumb_MCP_joint2: type revolute, parent L_thumb_proximal_base, child L_thumb_proximal, origin xyz=-0.0115 0.005 0.0034 rpy=0.9348037 -1.3508 0.1, axis -1 0 0, limit lower=0 upper=0.6248 effort=50 velocity=1
- added joint L_thumb_PIP_joint: type revolute, parent L_thumb_proximal, child L_thumb_intermediate, origin xyz=0 0.055863 -0.0039241 rpy=0.008299 0 0, axis -1 0 0, limit lower=0 upper=0.3578 effort=50 velocity=1, mimic joint=L_thumb_MCP_joint2 multiplier=1.1425 offset=0
- added joint R_index_DIP_joint: type revolute, parent R_index_proximal, child R_index_distal, origin xyz=0.001575 0.030445 0.010275 rpy=0.084288 0 0, axis 1 0 0, limit lower=0 upper=1.527 effort=50 velocity=1, mimic joint=R_index_MCP_joint multiplier=1.1169 offset=0
- added joint R_index_MCP_joint: type revolute, parent R_hand_base_link, child R_index_proximal, origin xyz=0.016376106 -0.000284483 -0.137082589 rpy=4.53 -0.034907 0, axis 1 0 0, limit lower=0 upper=1.41 effort=50 velocity=1
- added joint R_middle_DIP_joint: type revolute, parent R_middle_proximal, child R_middle_distal, origin xyz=0.0016673 0.030445 0.010275 rpy=0.111413 0 0, axis 1 0 0, limit lower=0 upper=1.527 effort=50 velocity=1, mimic joint=R_middle_MCP_joint multiplier=1.1169 offset=0
- added joint R_middle_MCP_joint: type revolute, parent R_hand_base_link, child R_middle_proximal, origin xyz=-0.001114894 -0.000284483 -0.137099589 rpy=4.524 0 0, axis 1 0 0, limit lower=0 upper=1.41 effort=50 velocity=1
- added joint R_pinky_DIP_joint: type revolute, parent R_pinky_proximal, child R_pinky_distal, origin xyz=0 0.030445 0.010275 rpy=0.002309 0 0, axis 1 0 0, limit lower=0 upper=1.527 effort=50 velocity=1, mimic joint=R_pinky_MCP_joint multiplier=1.1169 offset=0
- added joint R_pinky_MCP_joint: type revolute, parent R_hand_base_link, child R_pinky_proximal, origin xyz=-0.039300894 -0.000028483 -0.134262589 rpy=4.524 0.10472 0, axis 1 0 0, limit lower=0 upper=1.41 effort=50 velocity=1
- added joint R_ring_DIP_joint: type revolute, parent R_ring_proximal, child R_ring_distal, origin xyz=0 0.030445 0.010275 rpy=0.079748 0 0, axis 1 0 0, limit lower=0 upper=1.527 effort=50 velocity=1, mimic joint=R_ring_MCP_joint multiplier=1.1169 offset=0
- added joint R_ring_MCP_joint: type revolute, parent R_hand_base_link, child R_ring_proximal, origin xyz=-0.020288894 -0.000284483 -0.136176589 rpy=4.524 0.05236 0, axis 1 0 0, limit lower=0 upper=1.41 effort=50 velocity=1
- added joint R_thumb_DIP_joint: type revolute, parent R_thumb_intermediate, child R_thumb_distal, origin xyz=0 0.022558 -0.0020717 rpy=0.011642 0 0, axis 1 0 0, limit lower=0 upper=0.2775 effort=50 velocity=1, mimic joint=R_thumb_PIP_joint multiplier=0.7508 offset=0
- added joint R_thumb_MCP_joint1: type revolute, parent R_hand_base_link, child R_thumb_proximal_base, origin xyz=0.020450106 0.016955517 -0.071693589 rpy=4.7124 0 3.605907533, axis 0 -1 0, limit lower=0 upper=1.096 effort=50 velocity=1
- added joint R_thumb_MCP_joint2: type revolute, parent R_thumb_proximal_base, child R_thumb_proximal, origin xyz=-0.0115 -0.011843 0 rpy=5.21298075 1.5708 0, axis 1 0 0, limit lower=0 upper=0.6248 effort=50 velocity=1
- added joint R_thumb_PIP_joint: type revolute, parent R_thumb_proximal, child R_thumb_intermediate, origin xyz=0 0.055863 0.0039241 rpy=-0.008299 0 0, axis 1 0 0, limit lower=0 upper=0.3578 effort=50 velocity=1, mimic joint=R_thumb_MCP_joint2 multiplier=1.1425 offset=0
- joint left_hand_palm_joint: child left_hand_palm_link -> L_hand_base_link; origin xyz=0.0415 0.003 0 rpy=0 0 0 -> xyz=0.0415 0.003 0 rpy=0 -1.57 0
- joint right_hand_palm_joint: child right_hand_palm_link -> R_hand_base_link; origin xyz=0.0415 -0.003 0 rpy=0 0 0 -> xyz=0.0415 -0.003 0 rpy=0 -1.57 0
